Commit message: adding delay, randimization and noise

File: resources/robots/zq_humanoid/urdf/zq_sa01.urdf (robot description, URDF)
Before this commit: robot ZQ_Humanoid, 13 links, 12 joints
Links:
- removed link Base_link
- removed link Y1
- removed link Y2
- removed link Y3
- removed link Y4
- removed link Y5
- removed link Y6_foot
- removed link Z1
- removed link Z2
- removed link Z3
- removed link Z4
- removed link Z5
- removed link Z6_foot
- added link base_link, mass 10.176; collision box size=0.2 0.2 0.3; visual mesh filename=../meshes/Base_link.STL
- added link leg_l1_link, mass 1.6592; visual mesh filename=../meshes/LeftLeg_Link_01.STL
- added link leg_l2_link, mass 1.8008; visual mesh filename=../meshes/LeftLeg_Link_02.STL
- added link leg_l3_link, mass 3.9299; collision box size=0.08 0.08 0.25; visual mesh filename=../meshes/LeftLeg_Link_03.STL
- added link leg_l4_link, mass 2.72510; collision box size=0.05 0.05 0.28; visual mesh filename=../meshes/LeftLeg_Link_04.STL
- added link leg_l5_link, mass 0.16135; visual mesh filename=../meshes/LeftLeg_Link_05.STL
- added link leg_l6_link, mass 1.1926; collision mesh filename=../meshes/LeftLeg_Link_06.STL; visual mesh filename=../meshes/LeftLeg_Link_06.STL
- added link leg_r1_link, mass 1.6592; visual mesh filename=../meshes/RightLeg_Link_01.STL
- added link leg_r2_link, mass 1.8008; visual mesh filename=../meshes/RightLeg_Link_02.STL
- added link leg_r3_link, mass 3.9294; collision box size=0.08 0.08 0.25; visual mesh filename=../meshes/RightLeg_Link_03.STL
- added link leg_r4_link, mass 2.72497; collision box size=0.05 0.05 0.28; visual mesh filename=../meshes/RightLeg_Link_04.STL
- added link leg_r5_link, mass 0.16135; visual mesh filename=../meshes/RightLeg_Link_05.STL
- added link leg_r6_link, mass 1.1926; collision mesh filename=../meshes/RightLeg_Link_06.STL; visual mesh filename=../meshes/RightLeg_Link_06.STL
Joints:
- removed joint JOINT_Y1
- removed joint JOINT_Y2
- removed joint JOINT_Y3
- removed joint JOINT_Y4
- removed joint JOINT_Y5
- removed joint JOINT_Y6
- removed joint JOINT_Z1
- removed joint JOINT_Z2
- removed joint JOINT_Z3
- removed joint JOINT_Z4
- removed joint JOINT_Z5
- removed joint JOINT_Z6
- added joint leg_l1_joint: type revolute, parent base_link, child leg_l1_link, origin xyz=0 0.075 0 rpy=0 0 0, axis 1 0 0, limit lower=-0.523 upper=0.523 effort=140 velocity=25
- added joint leg_l2_joint: type revolute, parent leg_l1_link, child leg_l2_link, origin xyz=0 0 0 rpy=0 0 0, axis 0 0 1, limit lower=-0.3 upper=0.3 effort=140 velocity=25
- added joint leg_l3_joint: type revolute, parent leg_l2_link, child leg_l3_link, origin xyz=0 0 -0.1311 rpy=0 0 0, axis 0 1 0, limit lower=-1.204 upper=1.204 effort=140 velocity=25
- added joint leg_l4_joint: type revolute, parent leg_l3_link, child leg_l4_link, origin xyz=0 5.9998E-05 -0.3 rpy=0 0 0, axis 0 1 0, limit lower=0.0 upper=2.268 effort=140 velocity=25
- added joint leg_l5_joint: type revolute, parent leg_l4_link, child leg_l5_link, origin xyz=0 7.0122E-05 -0.37 rpy=0 0 0, axis 0 1 0, limit lower=-1.0 upper=0.6 effort=24 velocity=31
- added joint leg_l6_joint: type revolute, parent leg_l5_link, child leg_l6_link, origin xyz=0 0 0 rpy=0 0 0, axis 1 0 0, limit lower=-0.6 upper=0.6 effort=24 velocity=31
- added joint leg_r1_joint: type revolute, parent base_link, child leg_r1_link, origin xyz=0 -0.075 0 rpy=0 0 0, axis 1 0 0, limit lower=-0.523 upper=0.523 effort=140 velocity=25
- added joint leg_r2_joint: type revolute, parent leg_r1_link, child leg_r2_link, origin xyz=0 0 0 rpy=0 0 0, axis 0 0 1, limit lower=-0.3 upper=0.3 effort=140 velocity=25
- added joint leg_r3_joint: type revolute, parent leg_r2_link, child leg_r3_link, origin xyz=0 0 -0.1311 rpy=0 0 0, axis 0 1 0, limit lower=-1.204 upper=1.204 effort=140 velocity=25
- added joint leg_r4_joint: type revolute, parent leg_r3_link, child leg_r4_link, origin xyz=0 -5.9998E-05 -0.3 rpy=0 0 0, axis 0 1 0, limit lower=0.0 upper=2.268 effort=140 velocity=25
- added joint leg_r5_joint: type revolute, parent leg_r4_link, child leg_r5_link, origin xyz=0 -7.0122E-05 -0.37 rpy=0 0 0, axis 0 1 0, limit lower=-1.0 upper=0.6 effort=24 velocity=31
- added joint leg_r6_joint: type revolute, parent leg_r5_link, child leg_r6_link, origin xyz=0 0 0 rpy=0 0 0, axis 1 0 0, limit lower=-0.6 upper=0.6 effort=24 velocity=31
